Commit message: update

File: urdf/two_wheeled_robot_copy.urdf (robot description, URDF)
Before this commit: robot two_wheeled_robot, 9 links, 8 joints
Joints:
- joint camera_joint: origin xyz=0.305 0 0.08 rpy=0 0 0 -> xyz=0.08 0 0.3 rpy=0 0 0

Commit message: last

File: urdf/two_wheeled_robot_copy.urdf (robot description, URDF)
Before this commit: robot two_wheeled_robot, 9 links, 8 joints
Links:
- removed link imu_link
- removed link lidar_link
- link base_link: mass 15.0 -> 7.5; geometry collision box size=0.35 0.195 0.10; visual box size=0.35 0.195 0.10
- link drivewhl_l_link: geometry collision cylinder length=0.03 radius=0.07; visual cylinder length=0.03 radius=0.07
- link drivewhl_r_link: geometry collision cylinder length=0.03 radius=0.07; visual cylinder length=0.03 radius=0.07
- link front_caster: geometry collision sphere radius=0.0325; visual sphere radius=0.0325
Joints:
- removed joint imu_joint
- removed joint lidar_joint
- joint camera_joint: origin xyz=0.08 0 0.3 rpy=0 0 0 -> xyz=0.08 0 0.15 rpy=0 0 0
- joint caster_joint: origin xyz=0.217 0.0 -0.1 rpy=0 0 0 -> xyz=0.1 0.0 -0.1 rpy=0 0 0
- joint drivewhl_l_joint: origin xyz=-0.221 0.215 -0.05 rpy=0 0 0 -> xyz=-0.09 0.111 -0.05 rpy=0 0 0
- joint drivewhl_r_joint: origin xyz=-0.221 -0.215 -0.05 rpy=0 0 0 -> xyz=-0.09 -0.111 -0.05 rpy=0 0 0

Commit message: Jun 20

File: urdf/two_wheeled_robot_copy.urdf (robot description, URDF)
Before this commit: robot two_wheeled_robot, 7 links, 6 joints
Joints:
- joint camera_joint: origin xyz=0.08 0 0.15 rpy=0 0 0 -> xyz=0.0 0 0.2 rpy=0 0 0
